File: CAD/Soilsense/Soilsense.kicad_pcb (KiCad board)
At the start: 4 copper layers, 90 x 20 mm, 67 parts, among them J1 JLINK, Q1 MMBT3906, Q3 IRLML6401, SW1 B3U-1000P, U1 SHTC3, U2 nRF52833_QDxx, X1 KC3225K75.0000C1GE00, Y1 32MHz, Y2 32.768kHz

Commit message: NFC update
Parts:
- added L3: 4.7uH, inductor:L_Bourns_SDSS604A, F.Cu at (72.4, 44.8)
- J1: moved to B.Cu
- moved J1 34.7 mm to (80.3, 44.5), turned to -90 degrees
- moved C17 21.9 mm to (73.2, 48.6), turned to 180 degrees
- moved C18 19.8 mm to (71.3, 48.6), turned to 180 degrees
- moved U1 17.5 mm to (147.9, 57.0), turned to 0 degrees
- moved X1 11.8 mm to (96.2, 44.7), turned to 0 degrees
- moved Q3 7.34 mm to (92.2, 44.5), turned to 90 degrees
- moved D2 0.72 mm to (88.5, 45.5)
- moved C5 0.10 mm to (81.8, 59.1)
Routing:
- net Net-(U2-NFC2/P0.10): track 0.00 -> 18.3 mm
- net Net-(U2-NFC1/P0.09): track 0.00 -> 17.0 mm
- net GND: track 11.4 -> 13.4 mm, vias 4 -> 5
- net Net-(U2-XL1/P0.00): track 4.27 -> 5.51 mm
- net Net-(U2-XC2): track 4.40 -> 5.62 mm
- net Net-(U2-XC1): track 6.30 -> 7.50 mm
- net Net-(L1-Pad1): track 0.00 -> 1.17 mm
- net Net-(U2-XL2/P0.01): track 5.57 -> 6.69 mm
- added copper zone on F.Cu, net GND

Commit message: Layout
Parts:
- removed the U1 at (147.9, 57.0)
- removed the U1 at (72.2, 36.7)
- added D5: Zener Prot, Diode_SMD:D_SOD-523, F.Cu at (127.6, 51.0)
- added D6: Zener Prot, Diode_SMD:D_SOD-523, F.Cu at (101.5, 51.0)
- added Q2: Q_Photo_NPN, Soilsense:PHOTOTRANS_1708Metric, F.Cu at (88.1, 58.7)
- added R11: 10k, Resistor_SMD:R_0402_1005Metric, F.Cu at (91.7, 43.1)
- added R12: 10k, Resistor_SMD:R_0402_1005Metric, F.Cu at (93.6, 43.1)
- added TP11: NFC, TestPoint:TestPoint_Pad_D1.0mm, F.Cu at (73.1, 56.6)
- added U1: SHTC3, Sensor_Humidity:Sensirion_DFN-4-1EP_2x2mm_P1mm_EP0.7x1.6mm, F.Cu at (147.8, 57.2)
- C10: value 100n -> 1n
- C23: footprint Capacitor_SMD:C_0402_1005Metric -> Soilsense:C_0603_1608Metric
- D1, D2: value LL4148 -> CDSU101A; footprint Diode_SMD:D_MiniMELF -> Diode_SMD:D_SOD-523
- L6, L7: footprint Inductor_SMD:L_0402_1005Metric -> Soilsense:C_0603_1608Metric
- R9: footprint Resistor_SMD:R_0402_1005Metric -> Resistor_SMD:R_0603_1608Metric
- TP1: value 1.09 -> NFC
- moved TP10 84.2 mm to (49.3, 45.9)
- moved TP6 84.2 mm to (49.3, 33.7)
- moved TP7 84.2 mm to (49.3, 36.8)
- moved TP8 84.2 mm to (49.3, 39.8)
- moved TP9 84.2 mm to (49.3, 42.9)
- moved TP2 84.2 mm to (46.2, 36.8)
- moved TP3 84.2 mm to (46.2, 39.8)
- moved TP4 84.2 mm to (46.2, 42.9)
- moved TP5 84.2 mm to (46.2, 45.9)
- moved R6 73.0 mm to (145.5, 58.1), turned to -90 degrees
- moved R5 72.5 mm to (144.4, 58.1), turned to 90 degrees
- moved C2 72.2 mm to (145.7, 56.2), turned to 90 degrees
- moved TP1 50.1 mm to (73.1, 55.2), turned to 180 degrees
- moved RST1 38.9 mm to (87.8, 44.1)
- moved SW1 35.5 mm to (96.8, 57.4)
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Connections:
- net Net-(AE1-A) renamed /nRF52833_qdaa/RF_e
- net Net-(C21-Pad1) renamed /nRF52833_qdaa/RF_b
- net Net-(C23-Pad1) renamed /nRF52833_qdaa/RF_d
- net Net-(C23-Pad2) renamed /nRF52833_qdaa/RF_c
- net Net-(U2-ANT) renamed /nRF52833_qdaa/RF_a
- C10 pad 1: +3V6 -> SENS_OUT_HF_REF
- R9 pad 1: Net-(D4-A) -> Net-(X1-OUT)
- R9 pad 2: Net-(X1-OUT) -> Net-(D4-A)
- TP1 pad 1: 1.09 -> Net-(U2-NFC1/P0.09)
- U2 pad 35: BTN1 -> SENS_OUT_HF_REF
- U2 pad 6: 1.09 -> BTN1
Routing:
- net SENS_OUT_HF_REF: track 0.00 -> 6.36 mm
- net 1.09: track 3.55 -> 0.00 mm
- net Net-(U2-NFC1/P0.09): track 17.0 -> 20.1 mm
- net GND: track 13.4 -> 16.2 mm, vias 5 -> 9
- net BTN1: track 6.36 -> 3.55 mm
- net Net-(U2-NFC2/P0.10): track 18.3 -> 21.1 mm
- net /nRF52833_qdaa/RF_d: track 0.00 -> 2.60 mm
- net SENS_OUT: track 5.78 -> 7.98 mm
- net /nRF52833_qdaa/RF_c: track 0.00 -> 1.50 mm
- net PHOTO_OUT: track 5.70 -> 6.67 mm
- net Net-(U2-XC1): track 7.50 -> 6.94 mm
- net Net-(U2-XC2): track 5.62 -> 5.12 mm
- added copper zone on F.Cu, net /nRF52833_qdaa/RF_c
Other:
- board size 90 x 20 mm -> 91 x 21 mm
