File: CAD/Soilsense/Soilsense.kicad_sch (KiCad schematic)
At the start: 41 parts, among them J1 JLINK, Q1 MMBT3906, Q2 Q_Photo_NPN, Q3 IRLML6401, SW1 B3U-1000P, U1 SHTC3, X1 KC3225K75.0000C1GE00

Commit message: Layout
Parts:
- removed D1, D2: LL4148, Diode_SMD:D_MiniMELF, symbol Diode:LL4148
- removed TP1: 1.09, TestPoint:TestPoint_Pad_D1.0mm, symbol Connector:TestPoint
- added C10: 1n, Capacitor_SMD:C_0402_1005Metric, symbol Device:C_Small
- added D1, D2: CDSU101A, Diode_SMD:D_SOD-523, symbol Device:D_Schottky
- added D5, D6: Zener Prot, Diode_SMD:D_SOD-523, symbol Device:D_Schottky
- added R11, R12: 10k, Resistor_SMD:R_0402_1005Metric, symbol Device:R_Small_US
- Q2: footprint snapeda:TR8 -> Soilsense:PHOTOTRANS_1708Metric; LCSC C146233 -> (none); MPN (none) -> ALS-PT19-315C/L177/TR8
- R9: footprint Resistor_SMD:R_0402_1005Metric -> Resistor_SMD:R_0603_1608Metric
Connections:
- net +3V6: now also D2.1 (K)
- net CPARA: now also D1.2 (A), D5.1 (K)
- net GND: now also C10.2, D2.2 (A), D5.2 (A), D6.2 (A), R11.1
- net SENS_OUT: now also D1.1 (K)
- net at C3.1, Q3.2 (S), X1.1 (EN)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: now also R12.2
- net at X1.3 (OUT): now also R9.1; no longer R9.2
- net at D4.2 (A), H3.1: now also R9.2, D6.1 (K); no longer R9.1
- new net SENS_OUT_HF_REF: C10.1, R11.2, R12.1
Other:
- note added: "Smokey sacrificial Reverse current detector"
- note removed: "Audiovisual Reverse current detector"
- moved on the sheet: C4, D4, H3, R10
