File: CAD/Soilsense/nRF52833_qdaa.kicad_sch (KiCad schematic)
At the start: 29 parts, among them U2 nRF52833_QDxx, Y1 32MHz, Y2 32.768kHz

Commit message: NFC update
Parts:
- L3: footprint Inductor_SMD:L_Bourns-SRU8028_8.0x8.0mm -> inductor:L_Bourns_SDSS604A; MPN SDR0805-4R7ML -> SDR0604A-4R7ML

Commit message: Layout
Parts:
- removed C10: 100n, Capacitor_SMD:C_0402_1005Metric, symbol Device:C_Small
- added TP1, TP11: NFC, TestPoint:TestPoint_Pad_D1.0mm, symbol Connector:TestPoint
- C23: footprint Capacitor_SMD:C_0402_1005Metric -> Soilsense:C_0603_1608Metric
- L6, L7: footprint Inductor_SMD:L_0402_1005Metric -> Soilsense:C_0603_1608Metric
Connections:
- net at C17.2, L3.1, U2.22 (NFC1/P0.09): now also TP1.1
- net RF_a: now reaches C22.1, L5.2, U2.24 (ANT)
- net RF_e: now reaches AE1.1 (A), L7.1
- net at C18.1, L3.2, U2.23 (NFC2/P0.10): now also TP11.1
- net RF_b: now reaches C21.1, L4.2, L5.1
- net RF_d: now reaches C23.1, L6.1, L7.2
- net RF_c: now reaches C23.2, L4.1
Other:
- moved on the sheet: C11, C12, C13
