File: CAD/Soilsense_RFtest/Soilsense_RFtest.kicad_pcb (KiCad board)
At the start: 4 copper layers, 90 x 21 mm, 74 parts, among them J1 JLINK, Q1 MMBT3906, Q2 Q_Photo_NPN, Q3 IRLML6401, SW1 B3U-1000P, U1 SHTC3, U2 nRF52833_QDxx, X1 KC3225K75.0000C1GE00, Y1 32MHz, Y2 32.768kHz

Commit message: Small changes
Parts:
- removed C21: 1.2pF, Capacitor_SMD:C_0402_1005Metric
- removed L4: 2.2nH, Inductor_SMD:L_0402_1005Metric
- removed L5: 4.7nH, Inductor_SMD:L_0402_1005Metric
- added J2: Conn_Coaxial, Soilsense:U.FL_Hirose_U.FL-R-SMT-1_Vertical, F.Cu at (77.1, 59.0)
Routing:
- net GND: track 117.3 -> 119.9 mm, vias 240 -> 236
- net /nRF52833_qdaa/RF_b: track 1.86 -> 0.00 mm
- net /nRF52833_qdaa/RF_a: track 2.16 -> 1.38 mm
Other:
- board text added: "MINA SOILSENSE Rev 2.0 RF_BLANK"
- board text removed: "MINA SOILSENSE Rev 2.0"
