File: CAD/Soilsense_RFtest/nRF52833_qdaa.kicad_sch (KiCad schematic)
At the start: 30 parts, among them U2 nRF52833_QDxx, Y1 32MHz, Y2 32.768kHz

Commit message: Small changes
Parts:
- removed C21: 1.2pF, Capacitor_SMD:C_0402_1005Metric, symbol Device:C_Small
- removed L4: 2.2nH, Inductor_SMD:L_0402_1005Metric, symbol Device:L
- removed L5: 4.7nH, Inductor_SMD:L_0402_1005Metric, symbol Device:L
- added J2: Conn_Coaxial, Soilsense:U.FL_Hirose_U.FL-R-SMT-1_Vertical, symbol Connector:Conn_Coaxial
- C11, C12, C13, C15, C16, C19, C20, C22, C5, C6, C7, C8, C9, L1, TP1, TP11, U2, Y1, Y2: now not fitted
- L2: MPN MLG1005S15NHT000 -> (none); now not fitted
- L3: MPN SDR0604-4R7ML -> SDR0604A-4R7ML; now not fitted
Connections:
- net GND: now also J2.2 (Ext)
- net RF_c: now also J2.1 (In)
